Commit message: add boat model and disturbance on

File: urdf/simple_boat.urdf (robot description, URDF)
Before this commit: robot simple_boat, 3 links, 2 joints
Links:
- removed link left_wheel
- removed link right_wheel
- link base_link: mass 8.0 -> 12.0; geometry collision box size=0.9 0.42 0.20; visual box size=0.14 0.18 0.14
Joints:
- removed joint left_wheel_joint
- removed joint right_wheel_joint
